File: Hardware/KaraKuriSMD/SumibotSMD.kicad_sch (KiCad schematic)
At the start: 101 parts, among them J1 USB_B_Micro, M1 Left, M2 Right, Q1 DMG2301L, Q2 DMG2301L, Q3 DMG2301L, Q4 MBT3904DW1, Q5 DMG3406L, SW1 SW_SPDT, SW2 Reset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

Commit message: Aplique  jerarquía para trabajar en colaborativo
Parts:
- removed BT1: 2S, Connector_Molex:Molex_Micro-Latch_53253-0270_1x02_P2.00mm_Vertical, symbol Device:Battery
- removed BZ1: Buzzer, Buzzer_Beeper:Buzzer_Murata_PKMCS0909E, symbol Device:Buzzer
- removed C1, C13, C3, C4, C6, C7, C8, C9: 10uF, Capacitor_SMD:C_0805_2012Metric, symbol Device:C_Small
- removed C10, C12, C15, C18, C2, C20, C23: 0.1uF, Capacitor_SMD:C_0805_2012Metric, symbol Device:C_Small
- removed C11: 2.2nF, Capacitor_SMD:C_0805_2012Metric, symbol Device:C_Small
- removed C14: 10nF, Capacitor_SMD:C_0805_2012Metric, symbol Device:C_Small
- removed C16, C21: 47uF, Capacitor_SMD:C_0805_2012Metric, symbol Device:C_Polarized_Small
- removed C17, C22: 3.3nF, Capacitor_SMD:C_0805_2012Metric, symbol Device:C_Small
- removed C19, C24: 10uF, Capacitor_SMD:C_0805_2012Metric, symbol Device:C_Polarized_Small
- removed C5: 1uF, Capacitor_SMD:C_0805_2012Metric, symbol Device:C_Small
- removed D1: MBR1020VL, Diode_SMD:D_SOD-123F, symbol Diode:MBR1020VL
- removed D2: Done, LED_SMD:LED_0805_2012Metric_Pad1.15x1.40mm_HandSolder, symbol Device:LED
- removed D3, D4: LED, LED_SMD:LED_0805_2012Metric_Pad1.15x1.40mm_HandSolder, symbol Device:LED
- removed D5: Verde, LED_THT:LED_D5.0mm, symbol Device:LED
- removed D6: Amarillo, LED_THT:LED_D5.0mm, symbol Device:LED
- removed D7: Rojo, LED_THT:LED_D5.0mm, symbol Device:LED
- removed D8: 1N4151, Diode_SMD:D_0805_2012Metric, symbol Diode:1N4151
- removed D9: LED_RGBK, LED_SMD:LED_RGB_5050-6, symbol Device:LED_RGBK
- removed J1: USB_B_Micro, Connector_USB:USB_Micro-AB_Molex_47590-0001, symbol Connector:USB_B_Micro
- removed JP1, JP2, JP3, JP4, JP5: I2C Ad, Jumper:SolderJumper-3_P1.3mm_Bridged12_RoundedPad1.0x1.5mm, symbol Jumper:SolderJumper_3_Bridged12
- removed M1: Left, Connector_JST:JST_EH_S2B-EH_1x02_P2.50mm_Horizontal, symbol Motor:Motor_DC_ALT
- removed M2: Right, Connector_JST:JST_EH_S2B-EH_1x02_P2.50mm_Horizontal, symbol Motor:Motor_DC_ALT
- removed Q1, Q2, Q3: DMG2301L, Package_TO_SOT_SMD:SOT-23, symbol Transistor_FET:DMG2301L
- removed Q4: MBT3904DW1, Package_TO_SOT_SMD:SOT-363_SC-70-6, symbol Transistor_BJT:MBT3904DW1
- removed Q5: DMG3406L, Package_TO_SOT_SMD:SOT-23, symbol Transistor_FET:DMG3406L
- removed R1: 2M, Resistor_SMD:R_0805_2012Metric, symbol Device:R_US
- removed R10: 0, Resistor_SMD:R_0805_2012Metric, symbol Device:R_Small_US
- removed R11, R12, R19, R20, R28, R29, R3, R30, R31, R32, R8, R9: 1K, Resistor_SMD:R_0805_2012Metric, symbol Device:R_Small_US
- removed R13, R14: 100, Resistor_SMD:R_0805_2012Metric, symbol Device:R_Small_US
- removed R15, R16, R21: 1.5K, Resistor_SMD:R_0805_2012Metric, symbol Device:R_Small_US
- removed R17: 2.21K, Resistor_SMD:R_0805_2012Metric, symbol Device:R_Small_US
- removed R18, R27: 0.2, Resistor_SMD:R_0805_2012Metric, symbol Device:R_Small_US
- removed R2, R22, R23: 10K, Resistor_SMD:R_0805_2012Metric, symbol Device:R_Small_US
- removed R24, R25, R26: 3K, Resistor_SMD:R_0805_2012Metric, symbol Device:R_Small_US
- removed R33, R4, R5: 100K, Resistor_SMD:R_0805_2012Metric, symbol Device:R_Small_US
- removed R6: 1M, Resistor_SMD:R_0805_2012Metric, symbol Device:R_US
- removed R7: 2K, Resistor_SMD:R_0805_2012Metric, symbol Device:R_Small_US
- removed SW1: SW_SPDT, Button_Switch_SMD:SW_SPDT_PCM12, symbol Switch:SW_SPDT
- removed SW2: Reset, Button_Switch_SMD:SW_SPST_B3U-1000P, symbol Switch:SW_Push
- removed SW3: Boot, Button_Switch_SMD:SW_SPST_B3U-1000P, symbol Switch:SW_Push
- removed SW4: A, Button_Switch_SMD:SW_SPST_B3U-1000P, symbol Switch:SW_Push
- removed SW5: B, Button_Switch_SMD:SW_SPST_B3U-1000P, symbol Switch:SW_Push
- removed SW6: C, Button_Switch_SMD:SW_SPST_B3U-1000P, symbol Switch:SW_Push
- removed Serial1: 5V RX TX GND, Connector_PinHeader_2.54mm:PinHeader_1x04_P2.54mm_Vertical, symbol Connector_Generic:Conn_01x04
- removed U1: MCP73831-3-OT, Package_TO_SOT_SMD:SOT-23-5, symbol Battery_Management:MCP73831-3-OT
- removed U2: AP2112K-3.3, Package_TO_SOT_SMD:SOT-23-5, symbol Regulator_Linear:AP2112K-3.3
- removed U3: ESP32-WROOM-32, RF_Module:ESP32-WROOM-32, symbol RF_Module:ESP32-WROOM-32
- removed U4: MPU-9250, Sensor_Motion:InvenSense_QFN-24_3x3mm_P0.4mm, symbol Sensor_Motion:MPU-9250
- removed U5: LP2985-3.3, Package_TO_SOT_SMD:SOT-23-5, symbol Regulator_Linear:LP2985-3.3
- removed U6, U8: DRV8870DDA, Package_SO:Texas_HTSOP-8-1EP_3.9x4.9mm_P1.27mm_EP2.95x4.9mm_Mask2.4x3.1mm_ThermalVias, symbol Driver_Motor:DRV8870DDA
- removed U7: CH340C, Package_SO:SOIC-16_3.9x9.9mm_P1.27mm, symbol Interface_USB:CH340C
- removed i2C1: 5V GND SCL SDA, Connector_PinHeader_2.54mm:PinHeader_1x04_P2.54mm_Vertical, symbol Connector_Generic:Conn_01x04
Connections:
- no-connect marks 8 -> 0
Other:
- removed sheet Speaker
- added sheet Brain (SumibotBrain.kicad_sch)
- added sheet Motors (SumibotMotors.kicad_sch)
- added sheet OutPuts (OutPuts.kicad_sch)
- added sheet Power Management (Power Management.kicad_sch)
- added sheet Sensors (Sensors.kicad_sch)
- note removed: "600mA out 6V max in"
- note removed: "Auto Reset"
- note removed: "Driver y Motor"
- note removed: "Entrada y Cargador"
- note removed: "InPuts"
- note removed: "Inercial Sensor"
- note removed: "Interruptor y proteccion"
- note removed: "Microcontroller"
- note removed: "OutPuts"
- note removed: "Regulador"
- note removed: "USB"
- note removed: "V_USB - 6V Max +BATT Single Cell (4,2V Max)"
- title: KaraKuriSMD -> Sumibot
- moved on the sheet: H1, H2, H3, H4
