File: Hardware/Sumibot_V1/SumibotBrain.kicad_sch (KiCad schematic)
At the start: 28 parts, among them J1 USB_B_Micro, Q1 MBT3904DW1, SW1 Reset, SW2 Boot, U1 ESP32-WROOM-32, U2 CH340C

Commit message: implementó on/off toggle switch
Connections:
- net ON/OFF switch: now reaches U1.9 (IO33)
Changed lines of the file:
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@@
   (junction (at 75.692 172.847) (diameter 0) (color 0 0 0 0)
+  )
+  (junction (at 129.54 83.693) (diameter 0) (color 0 0 0 0)
   )
   (junction (at 75.692 214.757) (diameter 0) (color 0 0 0 0)
@@
     (stroke (width 0) (type default) (color 0 0 0 0))
   )
+  (wire (pts (xy 129.54 83.693) (xy 129.54 83.82))
+    (stroke (width 0) (type default) (color 0 0 0 0))
+  )
+  (wire (pts (xy 129.54 83.566) (xy 129.54 83.693))
+    (stroke (width 0) (type default) (color 0 0 0 0))
+  )
   (wire (pts (xy 157.734 187.071) (xy 157.734 188.976))
     (stroke (width 0) (type default) (color 0 0 0 0))
@@
   )
   (wire (pts (xy 75.692 214.757) (xy 79.375 214.757))
+    (stroke (width 0) (type default) (color 0 0 0 0))
+  )
+  (wire (pts (xy 133.35 83.82) (xy 129.54 83.82))
     (stroke (width 0) (type default) (color 0 0 0 0))
   )
@@
     (effects (font (size 1.27 1.27)) (justify left))
   )
+  (hierarchical_label "ON{slash}OFF switch" (shape bidirectional) (at 133.35 83.82 0)
+    (effects (font (size 1.27 1.27)) (justify left))
+  )
